Commit message: working IMU

File: src/my_robot_description/urdf/robot.urdf (robot description, URDF)
Before this commit: robot onshape, 21 links, 20 joints
Links:
- added link torso_imu, mass 0.01
Joints:
- added joint torso_to_imu: type fixed, parent torso, child torso_imu, origin xyz=0 0 0.1 rpy=0 0 0

Commit message: working force sensor!

File: src/my_robot_description/urdf/robot.urdf (robot description, URDF)
Before this commit: robot onshape, 22 links, 21 joints
Joints:
- joint left_hip_pitch: origin xyz=0.040849999999999969669 0.041699969999999995929 -0.01235999999999999252 rpy=-1.570796326794896558 0 1.570796326794896558 -> xyz=0.040849999999999969669 0.041699969999999968173 -0.01235999999999999252 rpy=-1.570796326794896558 0 1.570796326794896558
- joint left_hip_roll: origin xyz=-0.022849889999999997703 0.012500000000000004163 -0.022899000000000002686 rpy=-0 1.570796326794896336 0 -> xyz=-0.022849889999999987295 0.012500000000000004163 -0.022899000000000002686 rpy=-0 1.570796326794896336 0
